File: schema current.sch (EAGLE design)
At the start: 23 parts

Commit message: fixing all errors in schema
Parts:
- renumbered X1 to POWER
Connections:
- net MISO: now also MCP3008-CS1.MISO
- net MOSI: now also MCP3008-CS1.MOSI
- net SCL: now also 0X21.SCL, 0X22.SCL, 0X23.SCL, 0X24.SCL, 0X25.SCL, 0X26.SCL
- net SCLK: now also MCP3008-CS1.SCK
- net SDA: now also 0X21.SDA, 0X22.SDA, 0X23.SDA, 0X24.SDA, 0X25.SDA, 0X26.SDA
Changed lines of the file:
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@@
 <part name="GND8" library="supply1" deviceset="GND" device=""/>
 <part name="GND9" library="supply1" deviceset="GND" device=""/>
-<part name="X1" library="con-wago255" deviceset="233-102" device=""/>
+<part name="POWER" library="con-wago255" deviceset="233-102" device=""/>
 <part name="+3V5" library="supply1" deviceset="+3V3" device=""/>
 <part name="GND10" library="supply1" deviceset="GND" device=""/>
@@
 <instance part="GND8" gate="1" x="-81.28" y="58.42" rot="R180"/>
 <instance part="GND9" gate="1" x="-45.72" y="114.3"/>
-<instance part="X1" gate="G$1" x="-99.06" y="139.7"/>
+<instance part="POWER" gate="G$1" x="-99.06" y="139.7"/>
 <instance part="+3V5" gate="G$1" x="20.32" y="55.88"/>
 <instance part="GND10" gate="1" x="-12.7" y="48.26" rot="R180"/>
@@
 </segment>
 <segment>
-<pinref part="X1" gate="G$1" pin="-1"/>
+<pinref part="POWER" gate="G$1" pin="-1"/>
 <wire x1="-106.68" y1="139.7" x2="-106.68" y2="144.78" width="0.1524" layer="91"/>
 <pinref part="+3V1" gate="G$1" pin="+3V3"/>
@@
 </segment>
 <segment>
-<wire x1="55.88" y1="45.72" x2="55.88" y2="55.88" width="0.1524" layer="91"/>
-<label x="53.34" y="55.88" size="1.778" layer="95"/>
-</segment>
-<segment>
+<pinref part="0X24" gate="G$1" pin="SDA"/>
+<wire x1="-66.04" y1="45.72" x2="-66.04" y2="53.34" width="0.1524" layer="91"/>
+<label x="-68.58" y="53.34" size="1.778" layer="95"/>
+</segment>
+<segment>
+<pinref part="0X25" gate="G$1" pin="SDA"/>
 <wire x1="-5.08" y1="45.72" x2="-5.08" y2="53.34" width="0.1524" layer="91"/>
 <label x="-7.62" y="53.34" size="1.778" layer="95"/>
 </segment>
 <segment>
-<wire x1="-66.04" y1="45.72" x2="-66.04" y2="55.88" width="0.1524" layer="91"/>
-<label x="-68.58" y="55.88" size="1.778" layer="95"/>
-</segment>
-<segment>
-<wire x1="-55.88" y1="119.38" x2="-55.88" y2="121.92" width="0.1524" layer="91"/>
+<pinref part="0X26" gate="G$1" pin="SDA"/>
+<wire x1="55.88" y1="45.72" x2="55.88" y2="53.34" width="0.1524" layer="91"/>
+<label x="53.34" y="53.34" size="1.778" layer="95"/>
+</segment>
+<segment>
+<pinref part="0X23" gate="G$1" pin="SDA"/>
+<wire x1="127" y1="121.92" x2="127" y2="114.3" width="0.1524" layer="91"/>
+<label x="124.46" y="114.3" size="1.778" layer="95"/>
+</segment>
+<segment>
+<pinref part="0X22" gate="G$1" pin="SDA"/>
+<wire x1="66.04" y1="121.92" x2="66.04" y2="116.84" width="0.1524" layer="91"/>
+<label x="63.5" y="116.84" size="1.778" layer="95"/>
+</segment>
+<segment>
+<pinref part="0X21" gate="G$1" pin="SDA"/>
+<wire x1="5.08" y1="121.92" x2="5.08" y2="116.84" width="0.1524" layer="91"/>
+<label x="2.54" y="116.84" size="1.778" layer="95"/>
+</segment>
+<segment>
+<pinref part="0X20" gate="G$1" pin="SDA"/>
+<wire x1="-55.88" y1="121.92" x2="-55.88" y2="119.38" width="0.1524" layer="91"/>
 <label x="-58.42" y="119.38" size="1.778" layer="95"/>
-<pinref part="0X20" gate="G$1" pin="SDA"/>
-</segment>
-<segment>
-<wire x1="5.08" y1="111.76" x2="5.08" y2="121.92" width="0.1524" layer="91"/>
-<label x="5.08" y="111.76" size="1.778" layer="95"/>
-</segment>
-<segment>
-<wire x1="66.04" y1="111.76" x2="66.04" y2="121.92" width="0.1524" layer="91"/>
-<label x="66.04" y="109.22" size="1.778" layer="95"/>
-</segment>
-<segment>
-<wire x1="127" y1="111.76" x2="127" y2="121.92" width="0.1524" layer="91"/>
-<label x="127" y="111.76" size="1.778" layer="95"/>
 </segment>
 </net>
@@
 </segment>
 <segment>
-<wire x1="58.42" y1="45.72" x2="58.42" y2="55.88" width="0.1524" layer="91"/>
-<label x="58.42" y="55.88" size="1.778" layer="95"/>
-</segment>
-<segment>
+<pinref part="0X24" gate="G$1" pin="SCL"/>
+<wire x1="-63.5" y1="45.72" x2="-63.5" y2="53.34" width="0.1524" layer="91"/>
+<label x="-63.5" y="53.34" size="1.778" layer="95"/>
+</segment>
+<segment>
+<pinref part="0X25" gate="G$1" pin="SCL"/>
 <wire x1="-2.54" y1="45.72" x2="-2.54" y2="53.34" width="0.1524" layer="91"/>
 <label x="-2.54" y="53.34" size="1.778" layer="95"/>
 </segment>
 <segment>
-<wire x1="-63.5" y1="45.72" x2="-63.5" y2="55.88" width="0.1524" layer="91"/>
-<label x="-63.5" y="55.88" size="1.778" layer="95"/>
-</segment>
-<segment>
-<wire x1="-58.42" y1="119.38" x2="-58.42" y2="121.92" width="0.1524" layer="91"/>
+<pinref part="0X26" gate="G$1" pin="SCL"/>
+<wire x1="58.42" y1="45.72" x2="58.42" y2="53.34" width="0.1524" layer="91"/>
+<label x="58.42" y="53.34" size="1.778" layer="95"/>
+</segment>
+<segment>
+<pinref part="0X23" gate="G$1" pin="SCL"/>
+<wire x1="124.46" y1="121.92" x2="124.46" y2="114.3" width="0.1524" layer="91"/>
+<label x="119.38" y="114.3" size="1.778" layer="95"/>
+</segment>
+<segment>
+<pinref part="0X22" gate="G$1" pin="SCL"/>
+<wire x1="63.5" y1="121.92" x2="63.5" y2="116.84" width="0.1524" layer="91"/>
+<label x="58.42" y="116.84" size="1.778" layer="95"/>
+</segment>
+<segment>
+<pinref part="0X21" gate="G$1" pin="SCL"/>
+<wire x1="2.54" y1="121.92" x2="2.54" y2="116.84" width="0.1524" layer="91"/>
+<label x="-2.54" y="116.84" size="1.778" layer="95"/>
+</segment>
+<segment>
+<pinref part="0X20" gate="G$1" pin="SCL"/>
+<wire x1="-58.42" y1="121.92" x2="-58.42" y2="119.38" width="0.1524" layer="91"/>
 <label x="-63.5" y="119.38" size="1.778" layer="95"/>
-<pinref part="0X20" gate="G$1" pin="SCL"/>
-</segment>
-<segment>
-<wire x1="2.54" y1="111.76" x2="2.54" y2="121.92" width="0.1524" layer="91"/>
-<label x="-2.54" y="111.76" size="1.778" layer="95"/>
-</segment>
-<segment>
-<wire x1="63.5" y1="111.76" x2="63.5" y2="121.92" width="0.1524" layer="91"/>
-<label x="58.42" y="109.22" size="1.778" layer="95"/>
-</segment>
-<segment>
-<wire x1="124.46" y1="111.76" x2="124.46" y2="121.92" width="0.1524" layer="91"/>
-<label x="119.38" y="111.76" size="1.778" layer="95"/>
 </segment>
 </net>
@@
 <pinref part="MCP3008-CS0" gate="G$1" pin="MOSI"/>
 <wire x1="-58.42" y1="83.82" x2="-58.42" y2="81.28" width="0.1524" layer="91"/>
-<label x="-63.5" y="78.74" size="1.778" layer="95"/>
-</segment>
-<segment>
-<wire x1="2.54" y1="66.04" x2="2.54" y2="63.5" width="0.1524" layer="91"/>
-<label x="0" y="60.96" size="1.778" layer="95"/>
+<label x="-60.96" y="78.74" size="1.778" layer="95"/>
+</segment>
+<segment>
+<pinref part="MCP3008-CS1" gate="G$1" pin="MOSI"/>
+<wire x1="2.54" y1="66.04" x2="2.54" y2="60.96" width="0.1524" layer="91"/>
+<label x="0" y="58.42" size="1.778" layer="95"/>
 </segment>
 </net>
@@
 <segment>
 <pinref part="MCP3008-CS1" gate="G$1" pin="!CS"/>
-<wire x1="0" y1="66.04" x2="0" y2="63.5" width="0.1524" layer="91"/>
-<label x="-5.08" y="63.5" size="1.778" layer="95"/>
+<wire x1="0" y1="66.04" x2="0" y2="60.96" width="0.1524" layer="91"/>
+<label x="-5.08" y="60.96" size="1.778" layer="95"/>
 </segment>
 </net>
@@
 <wire x1="-55.88" y1="83.82" x2="-55.88" y2="81.28" width="0.1524" layer="91"/>
 <label x="-58.42" y="81.28" size="1.778" layer="95"/>
-<wire x1="-55.88" y1="83.82" x2="-55.88" y2="81.28" width="0.1524" layer="91"/>
-</segment>
-<segment>
-<wire x1="5.08" y1="66.04" x2="5.08" y2="63.5" width="0.1524" layer="91"/>
-<label x="2.54" y="63.5" size="1.778" layer="95"/>
+</segment>
+<segment>
+<pinref part="MCP3008-CS1" gate="G$1" pin="SCK"/>
+<wire x1="5.08" y1="66.04" x2="5.08" y2="60.96" width="0.1524" layer="91"/>
+<label x="2.54" y="60.96" size="1.778" layer="95"/>
 </segment>
 </net>
@@
 <net name="GND" class="0">
 <segment>
-<pinref part="X1" gate="G$1" pin="-2"/>
+<pinref part="POWER" gate="G$1" pin="-2"/>
 <wire x1="-106.68" y1="137.16" x2="-106.68" y2="132.08" width="0.1524" layer="91"/>
 <pinref part="GND3V3" gate="1" pin="GND"/>
@@
 <net name="MISO" class="0">
 <segment>
+<pinref part="RASPBERRY" gate="G$1" pin="B-4"/>
+<wire x1="165.1" y1="137.16" x2="154.94" y2="137.16" width="0.1524" layer="91"/>
+<label x="157.48" y="137.16" size="1.778" layer="95"/>
+</segment>
+<segment>
 <pinref part="MCP3008-CS0" gate="G$1" pin="MISO"/>
 <wire x1="-53.34" y1="83.82" x2="-53.34" y2="81.28" width="0.1524" layer="91"/>
@@
 </segment>
 <segment>
-<pinref part="RASPBERRY" gate="G$1" pin="B-4"/>
-<wire x1="165.1" y1="137.16" x2="154.94" y2="137.16" width="0.1524" layer="91"/>
-<label x="157.48" y="137.16" size="1.778" layer="95"/>
-</segment>
-<segment>
-<wire x1="7.62" y1="66.04" x2="7.62" y2="63.5" width="0.1524" layer="91"/>
-<label x="7.62" y="60.96" size="1.778" layer="95"/>
-</segment>
-</net>
+<pinref part="MCP3008-CS1" gate="G$1" pin="MISO"/>
+<wire x1="7.62" y1="66.04" x2="7.62" y2="60.96" width="0.1524" layer="91"/>
+<label x="7.62" y="58.42" size="1.778" layer="95"/>
+</segment>
+</net>
